Commit message: Replace robot model with UGV Belt Drive tracked model with sensors and physics

File: src/ugv_belt_drive/urdf/ugv_belt_drive_robot.urdf.xacro (robot description, xacro)
@@ -36,5 +36,4 @@
   <xacro:macro name="box_inertia" params="mass x y z">
     <inertial>
-      <origin xyz="0 0 -0.02" rpy="0 0 0"/>
       <mass value="${mass}"/>
       <inertia ixx="${mass/12.0*(y*y+z*z)}" ixy="0.0" ixz="0.0"
@@ -51,13 +50,4 @@
     </inertial>
   </xacro:macro>
-  <xacro:macro name="cylinder_inertia_y" params="mass r h">
-    <inertial>
-      <origin xyz="0 0 0" rpy="0 0 0"/>
-      <mass value="${mass}"/>
-      <inertia ixx="${mass/12.0*(3*r*r+h*h)}" ixy="0.0" ixz="0.0"
-               iyy="${mass*r*r/2.0}" iyz="0.0"
-               izz="${mass/12.0*(3*r*r+h*h)}"/>
-    </inertial>
-  </xacro:macro>
   <!-- ============================ BASE FOOTPRINT ========================= -->
   <link name="base_footprint"/>
@@ -78,5 +68,5 @@
       <geometry><box size="${chassis_length} ${chassis_width} ${chassis_height}"/></geometry>
     </collision>
-    <xacro:box_inertia mass="12.0" x="${chassis_length}" y="${chassis_width}" z="${chassis_height}"/>
+    <xacro:box_inertia mass="${chassis_mass}" x="${chassis_length}" y="${chassis_width}" z="${chassis_height}"/>
   </link>
   <!-- Yellow chassis trim strip (branding accent, purely cosmetic) -->
@@ -106,5 +96,5 @@
         <geometry><cylinder radius="${sprocket_radius}" length="${sprocket_width}"/></geometry>
       </collision>
-      <xacro:cylinder_inertia_y mass="${sprocket_mass}" r="${sprocket_radius}" h="${sprocket_width}"/>
+      <xacro:cylinder_inertia mass="${sprocket_mass}" r="${sprocket_radius}" h="${sprocket_width}"/>
     </link>
     <joint name="${side}_front_sprocket_joint" type="continuous">
@@ -126,5 +116,5 @@
         <geometry><cylinder radius="${sprocket_radius}" length="${sprocket_width}"/></geometry>
       </collision>
-      <xacro:cylinder_inertia_y mass="${sprocket_mass}" r="${sprocket_radius}" h="${sprocket_width}"/>
+      <xacro:cylinder_inertia mass="${sprocket_mass}" r="${sprocket_radius}" h="${sprocket_width}"/>
     </link>
     <joint name="${side}_rear_sprocket_joint" type="continuous">
@@ -135,6 +125,6 @@
       <dynamics damping="0.1" friction="0.05"/>
     </joint>
-    <!-- Belt shell: visual stadium shape spanning both sprockets.
-         Purely visual so rotating sprockets maintain 100% terrain traction. -->
+    <!-- Belt shell: visual-only stadium shape spanning both sprockets.
+         Collision uses a slim box so the belt still contacts terrain. -->
     <link name="${side}_belt">
       <visual>
@@ -143,4 +133,8 @@
         <material name="matte_black"/>
       </visual>
+      <collision>
+        <origin xyz="0 0 ${-ground_clearance}" rpy="0 0 0"/>
+        <geometry><box size="${track_wheelbase} ${sprocket_width} ${2*sprocket_radius*0.9}"/></geometry>
+      </collision>
       <inertial>
         <mass value="0.4"/>
@@ -582,14 +576,12 @@
       <wheel_separation>${track_separation}</wheel_separation>
       <wheel_radius>${sprocket_radius}</wheel_radius>
-      <max_wheel_torque>150.0</max_wheel_torque>
-      <max_wheel_acceleration>10.0</max_wheel_acceleration>
-      <max_linear_acceleration>5.0</max_linear_acceleration>
-      <max_angular_acceleration>6.0</max_angular_acceleration>
-      <max_linear_velocity>3.0</max_linear_velocity>
-      <min_linear_velocity>-3.0</min_linear_velocity>
-      <max_angular_velocity>4.0</max_angular_velocity>
-      <min_angular_velocity>-4.0</min_angular_velocity>
-      <topic>/ugv/cmd_vel</topic>
-      <odom_topic>/ugv/odom</odom_topic>
+      <max_linear_acceleration>3.0</max_linear_acceleration>
+      <max_angular_acceleration>4.0</max_angular_acceleration>
+      <max_linear_velocity>2.5</max_linear_velocity>
+      <min_linear_velocity>-2.5</min_linear_velocity>
+      <max_angular_velocity>3.0</max_angular_velocity>
+      <min_angular_velocity>-3.0</min_angular_velocity>
+      <topic>/cmd_vel</topic>
+      <odom_topic>/odom</odom_topic>
       <frame_id>odom</frame_id>
       <child_frame_id>base_footprint</child_frame_id>

Commit message: Fix UGV belt drive stability: remove dragging belt box, lower COM, and tune chassis mass

File: src/ugv_belt_drive/urdf/ugv_belt_drive_robot.urdf.xacro (robot description, xacro)
@@ -16,10 +16,10 @@
   <xacro:property name="chassis_width"  value="0.34"/>
   <xacro:property name="chassis_height" value="0.14"/>
-  <xacro:property name="chassis_mass"   value="9.0"/>
+  <xacro:property name="chassis_mass"   value="28.0"/>
   <xacro:property name="ground_clearance" value="0.07"/>
   <!-- Track / belt drive -->
   <xacro:property name="sprocket_radius" value="0.065"/>
   <xacro:property name="sprocket_width"  value="0.05"/>
-  <xacro:property name="sprocket_mass"   value="0.6"/>
+  <xacro:property name="sprocket_mass"   value="1.2"/>
   <xacro:property name="track_separation" value="0.40"/>      <!-- distance between left/right track centers -->
   <xacro:property name="track_wheelbase"  value="0.34"/>      <!-- distance between front and rear sprocket -->
@@ -36,4 +36,5 @@
   <xacro:macro name="box_inertia" params="mass x y z">
     <inertial>
+      <origin xyz="0 0 -0.03" rpy="0 0 0"/>
       <mass value="${mass}"/>
       <inertia ixx="${mass/12.0*(y*y+z*z)}" ixy="0.0" ixz="0.0"
@@ -125,6 +126,5 @@
       <dynamics damping="0.1" friction="0.05"/>
     </joint>
-    <!-- Belt shell: visual-only stadium shape spanning both sprockets.
-         Collision uses a slim box so the belt still contacts terrain. -->
+    <!-- Belt shell: visual representation spanning both sprockets. -->
     <link name="${side}_belt">
       <visual>
@@ -133,10 +133,6 @@
         <material name="matte_black"/>
       </visual>
-      <collision>
-        <origin xyz="0 0 ${-ground_clearance}" rpy="0 0 0"/>
-        <geometry><box size="${track_wheelbase} ${sprocket_width} ${2*sprocket_radius*0.9}"/></geometry>
-      </collision>
       <inertial>
-        <mass value="0.4"/>
+        <mass value="0.2"/>
         <inertia ixx="0.001" ixy="0" ixz="0" iyy="0.001" iyz="0" izz="0.001"/>
       </inertial>

Commit message: Fix Gazebo sprocket joint torque limits and add centerline avoidance for alternative valley routing

File: src/ugv_belt_drive/urdf/ugv_belt_drive_robot.urdf.xacro (robot description, xacro)
@@ -104,5 +104,6 @@
       <origin xyz="${track_wheelbase/2} ${y_sign*(track_separation/2)} ${-ground_clearance}" rpy="0 0 0"/>
       <axis xyz="0 1 0"/>
-      <dynamics damping="0.15" friction="0.05"/>
+      <limit effort="250.0" velocity="30.0"/>
+      <dynamics damping="0.05" friction="0.02"/>
     </joint>
     <!-- Rear (idler) sprocket -->
@@ -124,5 +125,6 @@
       <origin xyz="${-track_wheelbase/2} ${y_sign*(track_separation/2)} ${-ground_clearance}" rpy="0 0 0"/>
       <axis xyz="0 1 0"/>
-      <dynamics damping="0.1" friction="0.05"/>
+      <limit effort="250.0" velocity="30.0"/>
+      <dynamics damping="0.05" friction="0.02"/>
     </joint>
     <!-- Belt shell: visual representation spanning both sprockets. -->

Commit message: Lower Center of Mass to -0.06m and set spawn height to 2.70m for zero-impact upright settling

File: src/ugv_belt_drive/urdf/ugv_belt_drive_robot.urdf.xacro (robot description, xacro)
@@ -36,9 +36,9 @@
   <xacro:macro name="box_inertia" params="mass x y z">
     <inertial>
-      <origin xyz="0 0 -0.03" rpy="0 0 0"/>
+      <origin xyz="0 0 -0.06" rpy="0 0 0"/>
       <mass value="${mass}"/>
-      <inertia ixx="${mass/12.0*(y*y+z*z)}" ixy="0.0" ixz="0.0"
-               iyy="${mass/12.0*(x*x+z*z)}" iyz="0.0"
-               izz="${mass/12.0*(x*x+y*y)}"/>
+      <inertia ixx="${mass/12.0*(y*y+z*z) + 0.1}" ixy="0.0" ixz="0.0"
+               iyy="${mass/12.0*(x*x+z*z) + 0.1}" iyz="0.0"
+               izz="${mass/12.0*(x*x+y*y) + 0.2}"/>
     </inertial>
   </xacro:macro>
@@ -66,6 +66,6 @@
     </visual>
     <collision>
-      <origin xyz="0 0 0" rpy="0 0 0"/>
-      <geometry><box size="${chassis_length} ${chassis_width} ${chassis_height}"/></geometry>
+      <origin xyz="0 0 0.02" rpy="0 0 0"/>
+      <geometry><box size="${chassis_length*0.9} ${chassis_width*0.8} ${chassis_height*0.7}"/></geometry>
     </collision>
     <xacro:box_inertia mass="${chassis_mass}" x="${chassis_length}" y="${chassis_width}" z="${chassis_height}"/>

Commit message: Add SIH BOT mesh model and populate world with canyon blocks, boulders, and obstacles

File: src/ugv_belt_drive/urdf/ugv_belt_drive_robot.urdf.xacro (robot description, xacro)
@@ -61,6 +61,8 @@
   <link name="base_link">
     <visual>
-      <origin xyz="0 0 0" rpy="0 0 0"/>
-      <geometry><box size="${chassis_length} ${chassis_width} ${chassis_height}"/></geometry>
+      <origin xyz="0 0 -0.05" rpy="0 0 0"/>
+      <geometry>
+        <mesh filename="package://ugv_belt_drive/meshes/sih_bot.stl" scale="1.0 1.0 1.0"/>
+      </geometry>
       <material name="matte_black"/>
     </visual>

Commit message: Replace bot model with pure SIH BOT mesh and add intelligent 3D obstacle avoidance

File: src/ugv_belt_drive/urdf/ugv_belt_drive_robot.urdf.xacro (robot description, xacro)
@@ -73,11 +73,6 @@
     <xacro:box_inertia mass="${chassis_mass}" x="${chassis_length}" y="${chassis_width}" z="${chassis_height}"/>
   </link>
-  <!-- Yellow chassis trim strip (branding accent, purely cosmetic) -->
-  <link name="trim_strip">
-    <visual>
-      <geometry><box size="${chassis_length*0.9} 0.02 0.01"/></geometry>
-      <material name="signal_yellow"/>
-    </visual>
-  </link>
+  <!-- Yellow chassis trim strip -->
+  <link name="trim_strip"/>
   <joint name="trim_strip_joint" type="fixed">
     <parent link="base_link"/>
@@ -90,9 +85,4 @@
     <!-- Front (driven) sprocket -->
     <link name="${side}_front_sprocket">
-      <visual>
-        <origin xyz="0 0 0" rpy="${PI/2} 0 0"/>
-        <geometry><cylinder radius="${sprocket_radius}" length="${sprocket_width}"/></geometry>
-        <material name="dark_grey"/>
-      </visual>
       <collision>
         <origin xyz="0 0 0" rpy="${PI/2} 0 0"/>
@@ -111,9 +101,4 @@
     <!-- Rear (idler) sprocket -->
     <link name="${side}_rear_sprocket">
-      <visual>
-        <origin xyz="0 0 0" rpy="${PI/2} 0 0"/>
-        <geometry><cylinder radius="${sprocket_radius}" length="${sprocket_width}"/></geometry>
-        <material name="dark_grey"/>
-      </visual>
       <collision>
         <origin xyz="0 0 0" rpy="${PI/2} 0 0"/>
@@ -130,11 +115,6 @@
       <dynamics damping="0.05" friction="0.02"/>
     </joint>
-    <!-- Belt shell: visual representation spanning both sprockets. -->
+    <!-- Belt shell -->
     <link name="${side}_belt">
-      <visual>
-        <origin xyz="0 0 ${-ground_clearance}" rpy="0 0 0"/>
-        <geometry><box size="${track_wheelbase} ${sprocket_width+belt_thickness} ${2*sprocket_radius}"/></geometry>
-        <material name="matte_black"/>
-      </visual>
       <inertial>
         <mass value="0.2"/>
@@ -147,27 +127,9 @@
       <origin xyz="0 ${y_sign*(track_separation/2)} 0" rpy="0 0 0"/>
     </joint>
-    <!-- Transmission for the driven (front) sprocket -->
-    <xacro:if value="${driven}">
-      <transmission name="${side}_front_trans">
-        <type>transmission_interface/SimpleTransmission</type>
-        <joint name="${side}_front_sprocket_joint">
-          <hardwareInterface>hardware_interface/VelocityJointInterface</hardwareInterface>
-        </joint>
-        <actuator name="${side}_front_motor">
-          <hardwareInterface>hardware_interface/VelocityJointInterface</hardwareInterface>
-          <mechanicalReduction>1</mechanicalReduction>
-        </actuator>
-      </transmission>
-    </xacro:if>
   </xacro:macro>
   <xacro:track_side side="left"  y_sign="1"  driven="true"/>
   <xacro:track_side side="right" y_sign="-1" driven="true"/>
   <!-- ============================ ELECTRONICS ENCLOSURES ================= -->
-  <!-- Main compute + motor driver box -->
   <link name="electronics_box">
-    <visual>
-      <geometry><box size="0.16 0.20 0.06"/></geometry>
-      <material name="signal_yellow"/>
-    </visual>
     <collision>
       <geometry><box size="0.16 0.20 0.06"/></geometry>
@@ -182,8 +144,4 @@
   <!-- Battery pack -->
   <link name="battery_pack">
-    <visual>
-      <geometry><box size="0.18 0.10 0.06"/></geometry>
-      <material name="matte_black"/>
-    </visual>
     <collision>
       <geometry><box size="0.18 0.10 0.06"/></geometry>
