Commit message: Convert SIH BOT to DAE/OBJ and fix Gazebo mesh resource resolution

File: src/sih_bot/urdf/sih_bot.urdf.xacro (robot description, xacro)
@@ -27,5 +27,5 @@
       <origin xyz="0 0 -0.05" rpy="0 0 0"/>
       <geometry>
-        <mesh filename="package://sih_bot/meshes/sih_bot.stl" scale="1.0 1.0 1.0"/>
+        <mesh filename="package://sih_bot/meshes/sih_bot.dae" scale="1.0 1.0 1.0"/>
       </geometry>
       <material name="sih_charcoal"/>
@@ -47,6 +47,6 @@
     <visual>
       <material>
-        <ambient>0.2 0.22 0.26 1.0</ambient>
-        <diffuse>0.3 0.33 0.38 1.0</diffuse>
+        <ambient>0.25 0.28 0.32 1.0</ambient>
+        <diffuse>0.35 0.38 0.42 1.0</diffuse>
         <specular>0.6 0.6 0.6 1.0</specular>
       </material>

Commit message: Fix robot driving physics, wheel clearance, and state maintenance

File: src/sih_bot/urdf/sih_bot.urdf.xacro (robot description, xacro)
@@ -3,9 +3,9 @@
   <!-- ============================ CONSTANTS ============================== -->
   <xacro:property name="PI" value="3.1415926535897931"/>
-  <xacro:property name="robot_mass" value="28.0"/>
-  <xacro:property name="wheel_radius" value="0.065"/>
-  <xacro:property name="wheel_width" value="0.06"/>
+  <xacro:property name="robot_mass" value="25.0"/>
+  <xacro:property name="wheel_radius" value="0.075"/>
+  <xacro:property name="wheel_width" value="0.07"/>
   <xacro:property name="wheelbase" value="0.32"/>
-  <xacro:property name="track_width" value="0.36"/>
+  <xacro:property name="track_width" value="0.38"/>
   <!-- ============================ MATERIALS ============================== -->
   <material name="sih_charcoal">
@@ -20,5 +20,5 @@
     <parent link="base_footprint"/>
     <child link="base_link"/>
-    <origin xyz="0 0 ${wheel_radius + 0.015}" rpy="0 0 0"/>
+    <origin xyz="0 0 ${wheel_radius + 0.02}" rpy="0 0 0"/>
   </joint>
   <!-- ============================ CHASSIS (SIH BOT MESH) ================= -->
@@ -32,14 +32,14 @@
     </visual>
     <collision>
-      <origin xyz="0 0 0.04" rpy="0 0 0"/>
+      <origin xyz="0 0 0.08" rpy="0 0 0"/>
       <geometry>
-        <box size="0.48 0.38 0.28"/>
+        <box size="0.45 0.35 0.16"/>
       </geometry>
     </collision>
     <inertial>
       <!-- Lowered Center of Mass for rock-solid stability -->
-      <origin xyz="0 0 -0.06" rpy="0 0 0"/>
+      <origin xyz="0 0 -0.04" rpy="0 0 0"/>
       <mass value="${robot_mass}"/>
-      <inertia ixx="0.75" ixy="0.0" ixz="0.0" iyy="0.85" iyz="0.0" izz="1.10"/>
+      <inertia ixx="0.65" ixy="0.0" ixz="0.0" iyy="0.75" iyz="0.0" izz="0.95"/>
     </inertial>
   </link>
@@ -64,6 +64,6 @@
       <inertial>
         <origin xyz="0 0 0" rpy="0 0 0"/>
-        <mass value="1.2"/>
-        <inertia ixx="0.003" ixy="0" ixz="0" iyy="0.003" iyz="0" izz="0.005"/>
+        <mass value="1.5"/>
+        <inertia ixx="0.004" ixy="0" ixz="0" iyy="0.004" iyz="0" izz="0.007"/>
       </inertial>
     </link>
@@ -71,12 +71,12 @@
       <parent link="${parent}"/>
       <child link="${prefix}_wheel"/>
-      <origin xyz="${x_pos} ${y_pos} -0.015" rpy="0 0 0"/>
+      <origin xyz="${x_pos} ${y_pos} -0.02" rpy="0 0 0"/>
       <axis xyz="0 1 0"/>
-      <limit effort="300.0" velocity="30.0"/>
+      <limit effort="400.0" velocity="35.0"/>
       <dynamics damping="0.05" friction="0.02"/>
     </joint>
     <gazebo reference="${prefix}_wheel">
-      <mu1>1.8</mu1>
-      <mu2>1.8</mu2>
+      <mu1>2.5</mu1>
+      <mu2>2.5</mu2>
       <kp>1000000.0</kp>
       <kd>100.0</kd>

Commit message: Integrate Google Gemini Multimodal VLA Brain, dynamic API key support, and left/right obstacle avoidance reflexes

File: src/sih_bot/urdf/sih_bot.urdf.xacro (robot description, xacro)
@@ -77,6 +77,6 @@
     </joint>
     <gazebo reference="${prefix}_wheel">
-      <mu1>2.5</mu1>
-      <mu2>2.5</mu2>
+      <mu1>1.8</mu1>
+      <mu2>0.05</mu2>
       <kp>1000000.0</kp>
       <kd>100.0</kd>

File: src/ugv_belt_drive_ros2/urdf/ugv_belt_drive_robot.urdf.xacro (robot description, xacro)
@@ -105,6 +105,6 @@
     </joint>
     <gazebo reference="${side}_front_sprocket">
-      <mu1>2.5</mu1>
-      <mu2>2.5</mu2>
+      <mu1>1.8</mu1>
+      <mu2>0.05</mu2>
       <kp>1000000.0</kp>
       <kd>100.0</kd>
@@ -132,10 +132,10 @@
     </joint>
     <gazebo reference="${side}_rear_sprocket">
-      <mu1>2.5</mu1>
-      <mu2>2.5</mu2>
+      <mu1>1.8</mu1>
+      <mu2>0.05</mu2>
       <kp>1000000.0</kp>
       <kd>100.0</kd>
     </gazebo>
-    <!-- Track Belt Shell -->
+    <!-- Track Belt Shell (Visual only to avoid ground drag) -->
     <link name="${side}_belt">
       <visual>
@@ -144,10 +144,6 @@
         <material name="matte_black"/>
       </visual>
-      <collision>
-        <origin xyz="0 0 ${-ground_clearance}" rpy="0 0 0"/>
-        <geometry><box size="${track_wheelbase} ${sprocket_width} ${2*sprocket_radius*0.9}"/></geometry>
-      </collision>
       <inertial>
-        <mass value="0.4"/>
+        <mass value="0.2"/>
         <inertia ixx="0.001" ixy="0" ixz="0" iyy="0.001" iyz="0" izz="0.001"/>
       </inertial>
@@ -219,5 +215,5 @@
     <parent link="base_link"/>
     <child link="lidar_link"/>
-    <origin xyz="-0.04 0 ${chassis_height/2 + 0.05}" rpy="0 0 0"/>
+    <origin xyz="0.08 0 ${chassis_height/2 + 0.10}" rpy="0 0 0"/>
   </joint>
   <gazebo reference="lidar_link">
@@ -237,5 +233,5 @@
         </scan>
         <range>
-          <min>0.15</min>
+          <min>0.30</min>
           <max>25.0</max>
           <resolution>0.01</resolution>
