Commit message: fix(launch): streamline autonomous bringup, eliminate crashes and enable continuous navigation in Gazebo

File: src/ugv_belt_drive_ros2/urdf/ugv_belt_drive_robot.urdf.xacro (robot description, xacro)
@@ -64,6 +64,6 @@
     </visual>
     <collision>
-      <origin xyz="0 0 0" rpy="0 0 0"/>
-      <geometry><box size="${chassis_length} ${chassis_width} ${chassis_height}"/></geometry>
+      <origin xyz="0 0 0.03" rpy="0 0 0"/>
+      <geometry><box size="0.40 0.28 0.08"/></geometry>
     </collision>
     <xacro:box_inertia mass="${chassis_mass}" x="${chassis_length}" y="${chassis_width}" z="${chassis_height}"/>
@@ -421,17 +421,16 @@
   <!-- ============================ 4-SPROCKET SKID-STEER DRIVE ============= -->
   <gazebo>
+    <!-- Front Sprocket Drive System -->
     <plugin filename="gz-sim-diff-drive-system" name="gz::sim::systems::DiffDrive">
       <left_joint>left_front_sprocket_joint</left_joint>
-      <left_joint>left_rear_sprocket_joint</left_joint>
       <right_joint>right_front_sprocket_joint</right_joint>
-      <right_joint>right_rear_sprocket_joint</right_joint>
       <wheel_separation>${track_separation}</wheel_separation>
       <wheel_radius>${sprocket_radius}</wheel_radius>
-      <max_linear_acceleration>3.5</max_linear_acceleration>
-      <max_angular_acceleration>4.0</max_angular_acceleration>
-      <max_linear_velocity>2.0</max_linear_velocity>
-      <min_linear_velocity>-2.0</min_linear_velocity>
-      <max_angular_velocity>2.5</max_angular_velocity>
-      <min_angular_velocity>-2.5</min_angular_velocity>
+      <max_linear_acceleration>5.0</max_linear_acceleration>
+      <max_angular_acceleration>6.0</max_angular_acceleration>
+      <max_linear_velocity>2.5</max_linear_velocity>
+      <min_linear_velocity>-2.5</min_linear_velocity>
+      <max_angular_velocity>3.5</max_angular_velocity>
+      <min_angular_velocity>-3.5</min_angular_velocity>
       <topic>/cmd_vel</topic>
       <odom_topic>/odom</odom_topic>
@@ -440,30 +439,22 @@
       <odom_publish_frequency>50</odom_publish_frequency>
     </plugin>
+    <!-- Rear Sprocket Drive System -->
+    <plugin filename="gz-sim-diff-drive-system" name="gz::sim::systems::DiffDrive">
+      <left_joint>left_rear_sprocket_joint</left_joint>
+      <right_joint>right_rear_sprocket_joint</right_joint>
+      <wheel_separation>${track_separation}</wheel_separation>
+      <wheel_radius>${sprocket_radius}</wheel_radius>
+      <max_linear_acceleration>5.0</max_linear_acceleration>
+      <max_angular_acceleration>6.0</max_angular_acceleration>
+      <max_linear_velocity>2.5</max_linear_velocity>
+      <min_linear_velocity>-2.5</min_linear_velocity>
+      <max_angular_velocity>3.5</max_angular_velocity>
+      <min_angular_velocity>-3.5</min_angular_velocity>
+      <topic>/cmd_vel</topic>
+    </plugin>
     <plugin filename="gz-sim-joint-state-publisher-system" name="gz::sim::systems::JointStatePublisher">
       <topic>/joint_states</topic>
       <update_rate>30</update_rate>
     </plugin>
-    <plugin name="skid_steer_drive" filename="libgazebo_ros_diff_drive.so">
-      <ros><namespace>/ugv</namespace></ros>
-      <update_rate>50</update_rate>
-      <num_wheel_pairs>2</num_wheel_pairs>
-      <left_joint>left_front_sprocket_joint</left_joint>
-      <right_joint>right_front_sprocket_joint</right_joint>
-      <left_joint>left_rear_sprocket_joint</left_joint>
-      <right_joint>right_rear_sprocket_joint</right_joint>
-      <wheel_separation>${track_separation}</wheel_separation>
-      <wheel_separation>${track_separation}</wheel_separation>
-      <wheel_diameter>${2*sprocket_radius}</wheel_diameter>
-      <wheel_diameter>${2*sprocket_radius}</wheel_diameter>
-      <max_wheel_torque>28</max_wheel_torque>
-      <max_wheel_acceleration>2.5</max_wheel_acceleration>
-      <command_topic>cmd_vel</command_topic>
-      <odometry_topic>odom</odometry_topic>
-      <odometry_frame>odom</odometry_frame>
-      <robot_base_frame>base_footprint</robot_base_frame>
-      <publish_odom>true</publish_odom>
-      <publish_odom_tf>true</publish_odom_tf>
-      <publish_wheel_tf>true</publish_wheel_tf>
-    </plugin>
   </gazebo>
 </robot>

Commit message: Fix robot locomotion, multi-mission goal setting, dynamic obstacle bypass, and fast vectorized A* path planning

File: src/ugv_belt_drive_ros2/urdf/ugv_belt_drive_robot.urdf.xacro (robot description, xacro)
@@ -101,12 +101,12 @@
       <origin xyz="${track_wheelbase/2} ${y_sign*(track_separation/2)} ${-ground_clearance}" rpy="0 0 0"/>
       <axis xyz="0 1 0"/>
-      <limit effort="400.0" velocity="40.0"/>
-      <dynamics damping="0.05" friction="0.02"/>
+      <limit effort="1000.0" velocity="50.0"/>
+      <dynamics damping="0.01" friction="0.005"/>
     </joint>
     <gazebo reference="${side}_front_sprocket">
-      <mu1>1.8</mu1>
-      <mu2>0.05</mu2>
-      <kp>1000000.0</kp>
-      <kd>100.0</kd>
+      <mu1>2.0</mu1>
+      <mu2>2.0</mu2>
+      <kp>10000000.0</kp>
+      <kd>1.0</kd>
     </gazebo>
     <!-- Rear sprocket -->
@@ -128,12 +128,12 @@
       <origin xyz="${-track_wheelbase/2} ${y_sign*(track_separation/2)} ${-ground_clearance}" rpy="0 0 0"/>
       <axis xyz="0 1 0"/>
-      <limit effort="400.0" velocity="40.0"/>
-      <dynamics damping="0.05" friction="0.02"/>
+      <limit effort="1000.0" velocity="50.0"/>
+      <dynamics damping="0.01" friction="0.005"/>
     </joint>
     <gazebo reference="${side}_rear_sprocket">
-      <mu1>1.8</mu1>
-      <mu2>0.05</mu2>
-      <kp>1000000.0</kp>
-      <kd>100.0</kd>
+      <mu1>2.0</mu1>
+      <mu2>2.0</mu2>
+      <kp>10000000.0</kp>
+      <kd>1.0</kd>
     </gazebo>
     <!-- Track Belt Shell (Visual only to avoid ground drag) -->
@@ -421,16 +421,18 @@
   <!-- ============================ 4-SPROCKET SKID-STEER DRIVE ============= -->
   <gazebo>
-    <!-- Front Sprocket Drive System -->
+    <!-- Unified 4-Sprocket Skid-Steer Drive System -->
     <plugin filename="gz-sim-diff-drive-system" name="gz::sim::systems::DiffDrive">
       <left_joint>left_front_sprocket_joint</left_joint>
+      <left_joint>left_rear_sprocket_joint</left_joint>
       <right_joint>right_front_sprocket_joint</right_joint>
+      <right_joint>right_rear_sprocket_joint</right_joint>
       <wheel_separation>${track_separation}</wheel_separation>
       <wheel_radius>${sprocket_radius}</wheel_radius>
-      <max_linear_acceleration>5.0</max_linear_acceleration>
-      <max_angular_acceleration>6.0</max_angular_acceleration>
-      <max_linear_velocity>2.5</max_linear_velocity>
-      <min_linear_velocity>-2.5</min_linear_velocity>
-      <max_angular_velocity>3.5</max_angular_velocity>
-      <min_angular_velocity>-3.5</min_angular_velocity>
+      <max_linear_acceleration>10.0</max_linear_acceleration>
+      <max_angular_acceleration>12.0</max_angular_acceleration>
+      <max_linear_velocity>3.5</max_linear_velocity>
+      <min_linear_velocity>-3.5</min_linear_velocity>
+      <max_angular_velocity>4.5</max_angular_velocity>
+      <min_angular_velocity>-4.5</min_angular_velocity>
       <topic>/cmd_vel</topic>
       <odom_topic>/odom</odom_topic>
@@ -439,18 +441,4 @@
       <odom_publish_frequency>50</odom_publish_frequency>
     </plugin>
-    <!-- Rear Sprocket Drive System -->
-    <plugin filename="gz-sim-diff-drive-system" name="gz::sim::systems::DiffDrive">
-      <left_joint>left_rear_sprocket_joint</left_joint>
-      <right_joint>right_rear_sprocket_joint</right_joint>
-      <wheel_separation>${track_separation}</wheel_separation>
-      <wheel_radius>${sprocket_radius}</wheel_radius>
-      <max_linear_acceleration>5.0</max_linear_acceleration>
-      <max_angular_acceleration>6.0</max_angular_acceleration>
-      <max_linear_velocity>2.5</max_linear_velocity>
-      <min_linear_velocity>-2.5</min_linear_velocity>
-      <max_angular_velocity>3.5</max_angular_velocity>
-      <min_angular_velocity>-3.5</min_angular_velocity>
-      <topic>/cmd_vel</topic>
-    </plugin>
     <plugin filename="gz-sim-joint-state-publisher-system" name="gz::sim::systems::JointStatePublisher">
       <topic>/joint_states</topic>
